File: hardware/cm4_cb_use_v01/cm4-gpio.kicad_sch (KiCad schematic)
At the start: 15 parts, among them J1 DNP, J2 USB4105-GF-A, J3 SM04B-SRSS-TB(LF)(SN), U1 74LVC1G07SE-7

Commit message: New repo
Parts:
- removed J3: SM04B-SRSS-TB(LF)(SN), SM04B-SRSS-TB_LF__SN_:JST_SM04B-SRSS-TB(LF)(SN), symbol SM04B-SRSS-TB_LF__SN_:SM04B-SRSS-TB(LF)(SN)
- removed R3, R5: DNP, Resistor_SMD:R_0603_1608Metric_Pad0.98x0.95mm_HandSolder, symbol Device:R
Connections:
- no-connect marks 7 -> 6
Other:
- note removed: "I2C1_SCL"
- note removed: "I2C1_SDA"
- note removed: "Qwiic/Stemma"
- title: Raspberry Pi Compute Module 4 Base Carrier -> Compute Module 4 Carrierboard Utskytningsenhet
