File: hardware/cm4_cb_use_v01/cm4-gpio.kicad_sch (KiCad schematic)
At the start: 16 parts, among them J1 DNP, J4 molex_5046_2pin, J5 TPS62133RGTR, U1 SN74LVC1G07DCKR

Commit message: First draft done
Connections:
- net +3.3V: no longer Module1.86 (+3.3v_(Output))
- net +5V: now also J5.14 (VOS)
- net +7.4V: now reaches C1.1, C2.1, J4.1 (7,4V_VCC), J5.10 (AVIN), J5.11 (PVIN), J5.12 (PVIN), J5.13 (EN)
- net +1.8V: no longer names the net of Module1.88 (+1.8v_(Output))
- net +1.8V: no longer Module1.90 (+1.8v_(Output))
- no-connect marks 57 -> 60
Other:
- moved on the sheet: J4
Changed lines of the file:
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@@
   (junction (at 227.33 102.87) (diameter 1.016) (color 0 0 0 0))
   (junction (at 227.33 106.68) (diameter 1.016) (color 0 0 0 0))
+  (junction (at 236.22 77.47) (diameter 1.016) (color 0 0 0 0))
   (junction (at 241.3 77.47) (diameter 1.016) (color 0 0 0 0))
   (junction (at 254 77.47) (diameter 1.016) (color 0 0 0 0))
+  (no_connect (at 40.64 120.65))
   (no_connect (at 43.18 48.26))
   (no_connect (at 43.18 50.8))
@@
   (no_connect (at 43.18 144.78))
   (no_connect (at 43.18 147.32))
+  (no_connect (at 43.18 152.4))
+  (no_connect (at 43.18 154.94))
+  (no_connect (at 43.18 157.48))
   (no_connect (at 43.18 160.02))
   (no_connect (at 43.18 162.56))
@@
   (no_connect (at 104.14 167.64))
   (no_connect (at 104.14 170.18))
-  (no_connect (at 223.52 85.09))
   (no_connect (at 223.52 100.33))
   (wire (pts (xy 25.4 68.58) (xy 43.18 68.58))
@@
     (stroke (width 0) (type solid) (color 0 0 0 0))
   )
-  (wire (pts (xy 38.1 152.4) (xy 43.18 152.4))
-    (stroke (width 0) (type solid) (color 0 0 0 0))
-  )
-  (wire (pts (xy 38.1 154.94) (xy 43.18 154.94))
-    (stroke (width 0) (type solid) (color 0 0 0 0))
-  )
   (wire (pts (xy 40.64 45.72) (xy 40.64 53.34))
     (stroke (width 0) (type solid) (color 0 0 0 0))
@@
     (stroke (width 0) (type solid) (color 0 0 0 0))
   )
-  (wire (pts (xy 43.18 157.48) (xy 38.1 157.48))
-    (stroke (width 0) (type solid) (color 0 0 0 0))
-  )
   (wire (pts (xy 104.14 45.72) (xy 106.68 45.72))
     (stroke (width 0) (type solid) (color 0 0 0 0))
@@
     (stroke (width 0) (type solid) (color 0 0 0 0))
   )
+  (wire (pts (xy 163.83 81.28) (xy 166.37 81.28))
+    (stroke (width 0) (type solid) (color 0 0 0 0))
+  )
+  (wire (pts (xy 163.83 88.9) (xy 165.1 88.9))
+    (stroke (width 0) (type solid) (color 0 0 0 0))
+  )
+  (wire (pts (xy 165.1 88.9) (xy 165.1 111.76))
+    (stroke (width 0) (type solid) (color 0 0 0 0))
+  )
   (wire (pts (xy 166.37 30.48) (xy 166.37 26.67))
     (stroke (width 0) (type solid) (color 0 0 0 0))
@@
     (stroke (width 0) (type solid) (color 0 0 0 0))
   )
-  (wire (pts (xy 166.37 76.2) (xy 179.07 76.2))
-    (stroke (width 0) (type solid) (color 0 0 0 0))
-  )
-  (wire (pts (xy 166.37 83.82) (xy 167.64 83.82))
-    (stroke (width 0) (type solid) (color 0 0 0 0))
-  )
-  (wire (pts (xy 167.64 83.82) (xy 167.64 110.49))
+  (wire (pts (xy 173.99 76.2) (xy 179.07 76.2))
     (stroke (width 0) (type solid) (color 0 0 0 0))
   )
@@
     (stroke (width 0) (type solid) (color 0 0 0 0))
   )
+  (wire (pts (xy 223.52 85.09) (xy 236.22 85.09))
+    (stroke (width 0) (type solid) (color 0 0 0 0))
+  )
   (wire (pts (xy 223.52 90.17) (xy 241.3 90.17))
     (stroke (width 0) (type solid) (color 0 0 0 0))
@@
     (stroke (width 0) (type solid) (color 0 0 0 0))
   )
-  (wire (pts (xy 233.68 77.47) (xy 241.3 77.47))
+  (wire (pts (xy 233.68 77.47) (xy 236.22 77.47))
+    (stroke (width 0) (type solid) (color 0 0 0 0))
+  )
+  (wire (pts (xy 236.22 77.47) (xy 241.3 77.47))
+    (stroke (width 0) (type solid) (color 0 0 0 0))
+  )
+  (wire (pts (xy 236.22 85.09) (xy 236.22 77.47))
     (stroke (width 0) (type solid) (color 0 0 0 0))
   )
@@
     )
   )
-  (global_label "+3.3V" (shape output) (at 38.1 152.4 180)
-    (effects (font (size 1.27 1.27)) (justify right))
-    (property "Intersheet References" "${INTERSHEET_REFS}" (id 0) (at 0 2.54 0)
-      (effects (font (size 1.27 1.27)) hide)
-    )
-  )
-  (global_label "+1.8V" (shape output) (at 38.1 154.94 180)
-    (effects (font (size 1.27 1.27)) (justify right))
-    (property "Intersheet References" "${INTERSHEET_REFS}" (id 0) (at 0 0 0)
-      (effects (font (size 1.27 1.27)) hide)
-    )
-  )
-  (global_label "+1.8V" (shape output) (at 38.1 157.48 180)
-    (effects (font (size 1.27 1.27)) (justify right))
-    (property "Intersheet References" "${INTERSHEET_REFS}" (id 0) (at 0 2.54 0)
-      (effects (font (size 1.27 1.27)) hide)
-    )
-  )
   (global_label "+5V" (shape input) (at 109.22 142.24 0)
     (effects (font (size 1.27 1.27)) (justify left))
-    (property "Intersheet References" "${INTERSHEET_REFS}" (id 0) (at 0 0 0)
-      (effects (font (size 1.27 1.27)) hide)
+    (property "Intersheet References" "${INTERSHEET_REFS}" (id 0) (at 115.5036 142.1606 0)
+      (effects (font (size 1.27 1.27)) (justify left) hide)
     )
   )
@@
     (property "Intersheet References" "${INTERSHEET_REFS}" (id 0) (at -6.35 5.08 0)
       (effects (font (size 1.27 1.27)) hide)
+    )
+  )
+  (global_label "+7.4V" (shape output) (at 166.37 81.28 0)
+    (effects (font (size 1.27 1.27)) (justify left))
+    (property "Intersheet References" "${INTERSHEET_REFS}" (id 0) (at 174.4679 81.2006 0)
+      (effects (font (size 1.27 1.27)) (justify left) hide)
+    )
+  )
+  (global_label "+7.4V" (shape input) (at 173.99 76.2 180)
+    (effects (font (size 1.27 1.27)) (justify right))
+    (property "Intersheet References" "${INTERSHEET_REFS}" (id 0) (at 165.8921 76.1206 0)
+      (effects (font (size 1.27 1.27)) (justify right) hide)
     )
   )
@@
     (pin "1")
   )
-  (symbol (lib_id "power:GND") (at 167.64 110.49 0) (unit 1)
-    (in_bom yes) (on_board yes)
-    (property "Reference" "#PWR01" (id 0) (at 167.64 116.84 0)
-      (effects (font (size 1.27 1.27)) hide)
-    )
-    (property "Value" "GND" (id 1) (at 168.91 115.57 0))
-    (property "Footprint" "" (id 2) (at 167.64 110.49 0)
-      (effects (font (size 1.27 1.27)) hide)
-    )
-    (property "Datasheet" "" (id 3) (at 167.64 110.49 0)
+  (symbol (lib_id "power:GND") (at 165.1 111.76 0) (unit 1)
+    (in_bom yes) (on_board yes)
+    (property "Reference" "#PWR01" (id 0) (at 165.1 118.11 0)
+      (effects (font (size 1.27 1.27)) hide)
+    )
+    (property "Value" "GND" (id 1) (at 166.37 116.84 0))
+    (property "Footprint" "" (id 2) (at 165.1 111.76 0)
+      (effects (font (size 1.27 1.27)) hide)
+    )
+    (property "Datasheet" "" (id 3) (at 165.1 111.76 0)
       (effects (font (size 1.27 1.27)) hide)
     )
@@
     (pin "9")
   )
-  (symbol (lib_id "molex_5046_2pin:molex_5046_2pin") (at 154.94 72.39 0) (unit 1)
-    (in_bom yes) (on_board yes)
-    (property "Reference" "J4" (id 0) (at 161.29 71.12 0)
-      (effects (font (size 1.27 1.27)) (justify left))
-    )
-    (property "Value" "molex_5046_2pin" (id 1) (at 143.51 69.85 0)
-      (effects (font (size 1.27 1.27)) (justify left))
-    )
-    (property "Footprint" "Connector_Molex:Molex_KK-254_AE-6410-02A_1x02_P2.54mm_Vertical" (id 2) (at 154.94 69.85 0)
-      (effects (font (size 1.27 1.27)) hide)
-    )
-    (property "Datasheet" "https://no.rs-online.com/web/p/pcb-headers/6877269/?cm_mmc=NO-PLA-DS3A-_-google-_-CSS_NO_NO_Connectors_Whoop-_-(NO:Whoop!)+PCB+Headers+(3)-_-6877269&matchtype=&aud-828197004210:pla-388118817001&gclid=Cj0KCQiAyoeCBhCTARIsAOfpKxhvQcl0YpCa0uvFw0gKNlu5cbNg4HIXw8PskzbvxWI0hwQd_yhu1JYaAgmlEALw_wcB&gclsrc=aw.ds" (id 3) (at 158.75 67.31 0)
-      (effects (font (size 1.27 1.27)) hide)
-    )
-    (property "Coment" "Buy from RS" (id 4) (at 154.94 62.23 0)
-      (effects (font (size 1.27 1.27)) hide)
-    )
+  (symbol (lib_id "molex_5046_2pin:molex_5046_2pin") (at 152.4 77.47 0) (unit 1)
+    (in_bom yes) (on_board yes)
+    (property "Reference" "J4" (id 0) (at 158.75 76.2 0)
+      (effects (font (size 1.27 1.27)) (justify left))
+    )
+    (property "Value" "molex_5046_2pin" (id 1) (at 140.97 74.93 0)
+      (effects (font (size 1.27 1.27)) (justify left))
+    )
+    (property "Footprint" "Connector_Molex:Molex_KK-254_AE-6410-02A_1x02_P2.54mm_Vertical" (id 2) (at 152.4 74.93 0)
+      (effects (font (size 1.27 1.27)) hide)
+    )
+    (property "Datasheet" "https://no.rs-online.com/web/p/pcb-headers/6877269/?cm_mmc=NO-PLA-DS3A-_-google-_-CSS_NO_NO_Connectors_Whoop-_-(NO:Whoop!)+PCB+Headers+(3)-_-6877269&matchtype=&aud-828197004210:pla-388118817001&gclid=Cj0KCQiAyoeCBhCTARIsAOfpKxhvQcl0YpCa0uvFw0gKNlu5cbNg4HIXw8PskzbvxWI0hwQd_yhu1JYaAgmlEALw_wcB&gclsrc=aw.ds" (id 3) (at 156.21 72.39 0)
+      (effects (font (size 1.27 1.27)) hide)
+    )
+    (property "Coment" "Buy from RS" (id 4) (at 152.4 67.31 0)
+      (effects (font (size 1.27 1.27)) hide)
+    )

Commit message: updated
Parts:
- added R6: 262K, Resistor_SMD:R_0805_2012Metric, symbol Device:R
- added R7: 50K, Resistor_SMD:R_0805_2012Metric, symbol Device:R
- added SW1: SW_SPDT, c&k_slide_switch_1101M2S3AQE2:c&k_slide_switch_1101M2S3AQE2, symbol Switch:SW_SPDT
Connections:
- net +5V: now also R6.1
- net +7.4V: now also SW1.1 (A); no longer J4.1 (7,4V_VCC)
- net GND: now also R7.2; no longer J5.5 (FB)
- new net: J5.5 (FB), R6.2, R7.1
- new net: J4.1 (7,4V_VCC), SW1.2 (B)
Other:
- moved on the sheet: C1, C2, C3, C4, J4, J5, L1, R5
