File: hardware/cm4_cb_use_v01/cm4_cb_use_v01.kicad_sch (KiCad schematic)
At the start: 0 parts

Commit message: New repo
Other:
- title: Raspberry Pi Compute Module 4 Base Carrier -> Compute Module 4 Carrierboard Utskytningsenhet
Changed lines of the file:
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@@
-(kicad_sch (version 20201015) (generator eeschema)
-  (page 1 3)
+(kicad_sch (version 20210126) (generator eeschema)
   (paper "A4")
   (title_block
-    (title "Raspberry Pi Compute Module 4 Base Carrier")
+    (title "Compute Module 4 Carrierboard Utskytningsenhet")
     (date "2020-10-31")
     (rev "v01")
     (comment 2 "creativecommons.org/licenses/by-sa/4.0/")
     (comment 3 "License: CC BY-SA 4.0")
-    (comment 4 "Author: Shawn Hymel")
+    (comment 4 "Author: Martin Mæland")
   )
   (sheet (at 101.6 50.8) (size 38.1 38.1)
@@
       (reference "#PWR0108") (unit 1) (value "GND") (footprint "")
     )
-    (path "/fc4c71a5-1008-4ac4-98db-57c838c57d91/13ffbc3c-c167-4db3-adfc-fa2bdf2c4151"
-      (reference "#PWR0109") (unit 1) (value "GND") (footprint "")
-    )
     (path "/fc4c71a5-1008-4ac4-98db-57c838c57d91/b2bdacc5-5dd7-4aea-ae1d-b1028ef0bfb1"
       (reference "#PWR0110") (unit 1) (value "GND") (footprint "")
@@
       (reference "J2") (unit 1) (value "USB4105-GF-A") (footprint "USB4105-GF-A:GCT_USB4105-GF-A")
     )
-    (path "/fc4c71a5-1008-4ac4-98db-57c838c57d91/29b83231-3914-45e6-9ff5-265c2d7895d5"
-      (reference "J3") (unit 1) (value "SM04B-SRSS-TB(LF)(SN)") (footprint "SM04B-SRSS-TB_LF__SN_:JST_SM04B-SRSS-TB(LF)(SN)")
-    )
     (path "/fc4c71a5-1008-4ac4-98db-57c838c57d91/e653ed96-2ceb-42bc-905c-db47449cc067"
       (reference "JP1") (unit 1) (value "SolderJumper_2_Open") (footprint "Jumper:SolderJumper-2_P1.3mm_Open_RoundedPad1.0x1.5mm")
@@
       (reference "R2") (unit 1) (value "1k") (footprint "Resistor_SMD:R_0603_1608Metric_Pad0.98x0.95mm_HandSolder")
     )
-    (path "/fc4c71a5-1008-4ac4-98db-57c838c57d91/3016daa6-660f-43f1-af68-4db874e053a7"
-      (reference "R3") (unit 1) (value "DNP") (footprint "Resistor_SMD:R_0603_1608Metric_Pad0.98x0.95mm_HandSolder")
-    )
     (path "/fc4c71a5-1008-4ac4-98db-57c838c57d91/e581bea2-a554-4309-85f8-e6e0ce07520c"
       (reference "R4") (unit 1) (value "5.1k") (footprint "Resistor_SMD:R_0603_1608Metric_Pad0.98x0.95mm_HandSolder")
-    )
-    (path "/fc4c71a5-1008-4ac4-98db-57c838c57d91/9fa4a072-daf1-4573-89c6-c642e3ab4abe"
-      (reference "R5") (unit 1) (value "DNP") (footprint "Resistor_SMD:R_0603_1608Metric_Pad0.98x0.95mm_HandSolder")
     )
     (path "/fc4c71a5-1008-4ac4-98db-57c838c57d91/d38ddb23-f9c2-4a28-9fd8-d1fffee189f7"
@@
       (reference "#PWR0113") (unit 1) (value "GND") (footprint "")
     )
-    (path "/caa71f4c-454d-4ac9-b287-456eafb34991/59851573-5d3d-4fb7-a431-4d21e18e24d2"
-      (reference "#PWR0114") (unit 1) (value "GND") (footprint "")
+    (path "/caa71f4c-454d-4ac9-b287-456eafb34991/b2399ede-2d4f-433e-b8d4-681558150323"
+      (reference "#PWR?") (unit 1) (value "GND") (footprint "")
     )
-    (path "/caa71f4c-454d-4ac9-b287-456eafb34991/11143329-dd8d-4cc3-8fa4-452667b02f06"
-      (reference "#PWR0115") (unit 1) (value "GND") (footprint "")
-    )
-    (path "/caa71f4c-454d-4ac9-b287-456eafb34991/400cdc36-083c-4c59-a2cd-106a6a90acd8"
-      (reference "J4") (unit 1) (value "USB_OTG") (footprint "CM4IO:USB_Micro-B_EDAC_UCON00686")
+    (path "/caa71f4c-454d-4ac9-b287-456eafb34991/94c7d5d7-d648-439f-a208-c5670f7fe4ab"
+      (reference "J?") (unit 1) (value "1054500101") (footprint "Molex-1054500101-*")
     )
     (path "/caa71f4c-454d-4ac9-b287-456eafb34991/fafda8be-1326-444e-bcc1-8cb4aded3240"
       (reference "Module1") (unit 2) (value "ComputeModule4-CM4") (footprint "CM4IO:Raspberry-Pi-4-Compute-Module")
     )
-    (path "/caa71f4c-454d-4ac9-b287-456eafb34991/f98e44b3-cc4b-4d36-9b5b-fc739b8abd51"
-      (reference "R7") (unit 1) (value "2.2K 1%") (footprint "Resistor_SMD:R_0603_1608Metric_Pad0.98x0.95mm_HandSolder")
+    (path "/caa71f4c-454d-4ac9-b287-456eafb34991/396b9497-eaad-42f6-adc1-1d724e13ef1c"
+      (reference "R?") (unit 1) (value "2.2K 1%") (footprint "Resistor_SMD:R_0603_1608Metric_Pad0.98x0.95mm_HandSolder")
     )
-    (path "/caa71f4c-454d-4ac9-b287-456eafb34991/15a5dee6-171f-49e5-8d5e-d81e1c56a58d"
-      (reference "R8") (unit 1) (value "2.2K 1%") (footprint "Resistor_SMD:R_0603_1608Metric_Pad0.98x0.95mm_HandSolder")
+    (path "/caa71f4c-454d-4ac9-b287-456eafb34991/ceb61f80-9754-4184-938a-c0f30efebd07"
+      (reference "R?") (unit 1) (value "2.2K 1%") (footprint "Resistor_SMD:R_0603_1608Metric_Pad0.98x0.95mm_HandSolder")
     )
     (path "/caa71f4c-454d-4ac9-b287-456eafb34991/25c200c8-8d48-421b-ac68-c53b8df4e956"
