File: hardware/cm4_cb_use_v01/cm4_cb_use_v01.kicad_pcb (KiCad board)
At the start: 2 copper layers, 80 x 75 mm, 28 parts, among them J1 DNP, J2 HDMI_A, J3 1054500101, J4 molex_5046_2pin, J5 TPS62133RGTR, SW1 SW_SPDT, U1 SN74LVC1G07DCKR, U2 TPD2EUSB30

Commit message: made some mechanical drawings
Other:
- board text added: "Wireless Keepout"
Changed lines of the file:
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@@
   (gr_arc (start 80 120.000002) (end 76.5 120) (angle -90) (layer "Edge.Cuts") (width 0.1))
   (gr_line (start 80 123.5) (end 153 123.5) (layer "Edge.Cuts") (width 0.1))
+  (gr_text "Wireless\nKeepout" (at 112.5 100.1) (layer "Dwgs.User")
+    (effects (font (size 1 1) (thickness 0.25)))
+  )
+  (dimension (type aligned) (layer "Dwgs.User")
+    (pts (xy 76.499998 51.999998) (xy 156.5 52))
+    (height -18.199998)
+    (gr_text "80.0000 mm" (at 116.499999 32.000001 359.9999986) (layer "Dwgs.User")
+      (effects (font (size 1.5 1.5) (thickness 0.3)))
+    )
+    (format (units 3) (units_format 1) (precision 4))
+    (style (thickness 0.2) (arrow_length 1.27) (text_position_mode 0) (extension_height 0.58642) (extension_offset 0.5) keep_text_aligned)
+  )
+  (dimension (type aligned) (layer "Dwgs.User")
+    (pts (xy 153.000002 120) (xy 153 52))
+    (height 14.799999)
+    (gr_text "68.0000 mm" (at 169.6 86 -89.99999831) (layer "Dwgs.User")
+      (effects (font (size 1.5 1.5) (thickness 0.3)))
+    )
+    (format (units 3) (units_format 1) (precision 4))
+    (style (thickness 0.2) (arrow_length 1.27) (text_position_mode 0) (extension_height 0.58642) (extension_offset 0.5) keep_text_aligned)
+  )
+  (dimension (type aligned) (layer "Dwgs.User")
+    (pts (xy 153 52) (xy 79.999998 52))
+    (height 10.699999)
+    (gr_text "73.0000 mm" (at 116.499999 39.500001) (layer "Dwgs.User")
+      (effects (font (size 1.5 1.5) (thickness 0.3)))
+    )
+    (format (units 3) (units_format 1) (precision 4))
+    (style (thickness 0.2) (arrow_length 1.27) (text_position_mode 0) (extension_height 0.58642) (extension_offset 0.5) keep_text_aligned)
+  )
+  (dimension (type aligned) (layer "Dwgs.User")
+    (pts (xy 153 48.5) (xy 153.000002 123.499998))
+    (height -27.699998)
+    (gr_text "75.0000 mm" (at 182.499999 85.999998 270.0000015) (layer "Dwgs.User")
+      (effects (font (size 1.5 1.5) (thickness 0.3)))
+    )
+    (format (units 3) (units_format 1) (precision 4))
+    (style (thickness 0.2) (arrow_length 1.27) (text_position_mode 0) (extension_height 0.58642) (extension_offset 0.5) keep_text_aligned)
+  )
+  (dimension (type leader) (layer "Dwgs.User")
+    (pts (xy 153 52) (xy 164.5 43.6))
+    (gr_text "4xM3" (at 170.5 43.6) (layer "Dwgs.User")
+      (effects (font (size 1.5 1.5) (thickness 0.3)))
+    )
+    (format (units 0) (units_format 0) (precision 4) (override_value "4xM3"))
+    (style (thickness 0.2) (arrow_length 1.27) (text_position_mode 0) (text_frame 0) (extension_offset 0.5))
+  )
   (segment (start 119.5 90.4) (end 119.5 112.08) (width 0.2) (layer "F.Cu") (net 1))
   (segment (start 131.92 79.1) (end 130.8 79.1) (width 0.2) (layer "F.Cu") (net 1))
